File: Electronics/PowerDistribution/PowerDistribution.kicad_pcb (KiCad board)
At the start: 2 copper layers, 50 x 45 mm, 25 parts, among them J1 Screw_Terminal_01x02, J2 Conn_02x03_Odd_Even, J3 Conn_02x03_Odd_Even, J4 USB_A_Double, J5 Screw_Terminal_01x02, P1 R-78Bxx-2.0, Q1 BS170

Commit message: [Electronics] PCB - first complete version.
Parts:
- removed D3: LED, LEDs:LED_D5.0mm
- removed I1: BD4xxxG, MiAM:SSOP-5
- removed Q1: BS170, TO_SOT_Packages_THT:TO-92_Molded_Narrow
- removed R3: 100k, Resistors_THT:R_Axial_DIN0207_L6.3mm_D2.5mm_P10.16mm_Horizontal
- removed R4: 2k, Resistors_THT:R_Axial_DIN0207_L6.3mm_D2.5mm_P10.16mm_Horizontal
- removed RV1: 50k, Potentiometers:Potentiometer_Trimmer_Vishay_T73YP_Horizontal
- added C6: CP1, Capacitor_THT:CP_Radial_D5.0mm_P2.50mm, F.Cu at (120.5, 88.0)
- added J6: Conn_01x01_Male, Connector_PinHeader_2.54mm:PinHeader_1x01_P2.54mm_Vertical, F.Cu at (119.5, 83.5)
- added J7: Conn_02x02_Odd_Even, Connector_PinHeader_2.54mm:PinHeader_2x02_P2.54mm_Vertical, F.Cu at (103.0, 73.0)
- added P2: R-78Bxx-2.0, MiAM:CONV_R-78Bxx-2.0, F.Cu at (110.5, 78.0)
- C5: footprint Capacitors_THT:CP_Radial_D5.0mm_P2.50mm -> Capacitor_THT:CP_Radial_D5.0mm_P2.50mm
- D1, D2: footprint LEDs:LED_D5.0mm -> LED_THT:LED_D5.0mm
- J1, J5: footprint Connectors:bornier2 -> TerminalBlock:TerminalBlock_bornier-2_P5.08mm
- J2, J3: footprint Pin_Headers:Pin_Header_Straight_2x03_Pitch2.54mm -> Connector_PinHeader_2.54mm:PinHeader_2x03_P2.54mm_Vertical
- R1, R2: footprint Resistors_THT:R_Axial_DIN0207_L6.3mm_D2.5mm_P10.16mm_Horizontal -> Resistor_THT:R_Axial_DIN0207_L6.3mm_D2.5mm_P10.16mm_Horizontal
- moved R1 7.72 mm to (138.0, 87.5)
- moved R2 3.04 mm to (141.0, 81.0)
- moved C5 2.15 mm to (114.5, 88.0), turned to 270 degrees
- moved P1 1.68 mm to (127.5, 83.0)
Connections:
- C2 pad 3: (no net) -> Net-(C2-Pad3)
- J4 pad 2: (no net) -> Net-(J4-Pad2)
- J4 pad 3: (no net) -> Net-(J4-Pad3)
- J4 pad 5: (no net) -> Net-(J4-Pad5)
- J4 pad 6: (no net) -> Net-(J4-Pad6)
Routing:
- net Net-(J7-Pad1): track 0.00 -> 12.6 mm
- net Net-(D1-Pad2): track 0.00 -> 11.0 mm
- net Net-(D2-Pad2): track 0.00 -> 8.34 mm
- added copper zone on F.Cu, net +12V
- added copper zone on B.Cu, net GND
- added copper zone on F.Cu, net Net-(C1-Pad1)
- added copper zone on F.Cu, net Net-(J3-Pad1)
Other:
- board size 50 x 45 mm -> 50 x 40 mm
- net class Default: clearance 0.2 -> 0.4; trace_width 0.25 -> 0.4
- rule trace_clearance: 0.2 -> 0.4
